File: hw-openmower-utils-satabob/hw-openmower-utils-satabob.kicad_pcb (KiCad board)
At the start: 2 copper layers, 40.9 x 66.5 mm, 4 parts, among them J1 67800-8005, J2 Conn_01x20_Pin, J3 Conn_01x20_Pin, U1 Pico

Commit message: added git version to pcb
Other:
- board text added: "${git_version}"
- board text removed: "v1.0 rev A"
Changed lines of the file:
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@@
 		)
 	)
+	(property "git_version" "v0.0.0")
 	(net 0 "")
 	(net 1 "GND")
@@
 		(tags "Connector")
 		(property "Reference" "J1"
-			(at -3.81 -0.925 360)
+			(at -3.81 -0.925 0)
 			(layer "F.SilkS")
 			(hide yes)
@@
 		)
 		(property "Value" "67800-8005"
-			(at -3.81 -0.925 360)
+			(at -3.81 -0.925 0)
 			(layer "F.SilkS")
 			(hide yes)
@@
 		)
 		(fp_text user "${REFERENCE}"
-			(at -3.81 -0.925 360)
+			(at -3.81 -0.925 0)
 			(layer "F.Fab")
 			(effects
@@
 		(layer "Edge.Cuts")
 	)
-	(gr_text "v1.0 rev A"
+	(gr_text "${git_version}"
 		(at 110 36 180)
 		(layer "B.Cu")
@@
 		)
 	)
+	(gr_text "${git_version}"
+		(at 148.7 47.3 90)
+		(layer "F.SilkS")
+		(effects
+			(font
+				(size 1 1)
+				(thickness 0.1)
+			)
+			(justify left bottom)
+		)
+	)
 	(gr_text "Sata Breakout"
-		(at 149.3 47.4 90)
+		(at 147.1 47.4 90)
 		(layer "F.SilkS")
 		(effects
@@
 	)
 	(gr_text "OpenMower"
-		(at 147.5 45.9 90)
+		(at 145.3 45.9 90)
 		(layer "F.SilkS")
 		(effects
